File: hardware/radio_xcvr.sch (KiCad schematic (older format))
At the start: 37 parts, among them J3 SMA, U2 MAX7032ATJ+, Y1 17.63416MHz, 4.5pF load cap., Y2 SFECV10M7JA00

Commit message: Schematic checklist
Parts:
- C10, C11, C12, C13, C14, C15, C16, C17, C18, C19, C20, C21, C22, C23, C24, C25, C26, C27, C28, C29, C30, C6, C7, C8, C9: footprint (none) -> link-434:C_0402_1005Metric
- J3: footprint (none) -> link-434:SMA_Linx_CONSMA001_Vertical; Link (none) -> https://www.mouser.at/ProductDetail/Linx-Technologies/CONSM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; MPN (none) -> CONSMA001-C-G
- L1, L2, L4: footprint (none) -> link-434:L_Coilcraft_0603CS; Link (none) -> https://www.mouser.at/ProductDetail/Coilcraft/0603CS-22NXJLW; MPN (none) -> 0603CS-22NXJLW
- L3: footprint (none) -> link-434:L_Coilcraft_0603CS; Link (none) -> https://www.mouser.at/ProductDetail/Coilcraft/0603CS-68NXJLW; MPN (none) -> 0603CS-68NXJLW
- L5: footprint (none) -> link-434:L_Coilcraft_0603CS; Link (none) -> https://www.mouser.at/ProductDetail/Coilcraft/0603CS-10NXJLU; MPN (none) -> 0603CS-10NXJLU
- L6: footprint (none) -> link-434:L_Murata_LQW18ASxxxx00x; Link (none) -> https://www.mouser.at/ProductDetail/Murata-Electronics/LQW1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; MPN (none) -> LQW18AS16NJ00D
- R16, R17: footprint (none) -> link-434:R_0402_1005Metric
- U2: footprint (none) -> link-434:QFN-32-1EP_5x5mm_P0.5mm_EP3.1x3.1mm_ThermalVias; Link (none) -> https://www.mouser.at/ProductDetail/Maxim-Integrated/MAX703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; MPN (none) -> MAX7032ATJ+
- Y1: footprint (none) -> link-434:Crystal_SMD_HC49-SD; Link (none) -> https://www.mouser.at/ProductDetail/Crystek-Corporation/017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; MPN (none) -> 017301
- Y2: footprint (none) -> link-434:Resonator_SMD_muRata_SFECV-3Pin_6.9x2.9mm; Link (none) -> https://www.mouser.at/ProductDetail/Murata-Electronics/SFEC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; MPN (none) -> SFECV10M7JA00-R0
